File: rpipico.kicad_pcb (KiCad board)
At the start: 2 copper layers, 21.2 x 29.1 mm, 34 parts, among them J1 USB_C_Receptacle_USB2.0, J2 Conn_01x02_Pin, J3 Conn_01x13, J4 Conn_01x13, J5 Conn_01x04, J6 Conn_01x03, J7 Conn_01x04, J8 Conn_01x02, U2 W25Q128JVS, U3 RP2040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

Commit message: Add files via upload
Parts:
- added J9: Conn_01x02, Connector_PinHeader_1.00mm:PinHeader_1x02_P1.00mm_Vertical, F.Cu at (132.3, 90.5)
- moved C3 1.08 mm to (144.7, 86.6)
- moved C4 1.08 mm to (145.5, 86.6)
- moved C5 0.99 mm to (143.0, 86.6)
- moved C6 0.99 mm to (143.9, 86.6)
- moved J2 0.82 mm to (134.3, 89.5)
- moved R5 0.66 mm to (134.5, 88.0), turned to 0 degrees
- moved C9 0.47 mm to (135.8, 88.2)
- moved C10 0.34 mm to (136.6, 88.2)
- moved C13 0.11 mm to (140.5, 86.6)
Connections:
- U3 pad 26: unconnected-(U3-RUN-Pad26) -> Net-(J9-Pin_2)
Routing:
- net Net-(J9-Pin_2): track 0.00 -> 15.4 mm, vias 0 -> 1
- net GND: track 39.3 -> 42.2 mm, vias 12 -> 11
- net /QSPI_SS: track 10.5 -> 9.16 mm
- net Net-(J4-Pin_2): track 15.8 -> 16.7 mm
- net Net-(J4-Pin_3): track 15.9 -> 16.8 mm
- net Net-(J3-Pin_13): track 14.2 -> 15.2 mm
- net Net-(J4-Pin_1): track 15.7 -> 16.6 mm
- net Net-(J2-Pin_1): track 2.63 -> 1.81 mm
- net +3.3V: track 67.3 -> 66.6 mm

Commit message: Add files via upload
Routing:
- net Net-(J9-Pin_2): track 15.4 -> 14.7 mm
Changed lines of the file:
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@@
   (segment (start 142.9 94.706299) (end 142.9 95.0125) (width 0.1) (layer "F.Cu") (net 12))
   (via (at 138.7 94.077592) (size 0.6) (drill 0.4) (layers "F.Cu" "B.Cu") (net 12))
-  (segment (start 132.195 89.5) (end 132.325 89.5) (width 0.1) (layer "B.Cu") (net 12))
-  (segment (start 131.5 90.195) (end 132.195 89.5) (width 0.1) (layer "B.Cu") (net 12))
-  (segment (start 134.1066 94.0816) (end 131.5 91.475) (width 0.1) (layer "B.Cu") (net 12))
-  (segment (start 131.5 91.475) (end 131.5 90.195) (width 0.1) (layer "B.Cu") (net 12))
-  (segment (start 138.695992 94.0816) (end 134.1066 94.0816) (width 0.1) (layer "B.Cu") (net 12))
-  (segment (start 138.7 94.077592) (end 138.695992 94.0816) (width 0.1) (layer "B.Cu") (net 12))
+  (segment (start 132.96 89.53396) (end 132.92604 89.5) (width 0.1) (layer "B.Cu") (net 12))
+  (segment (start 132.96 92.405) (end 132.96 89.53396) (width 0.1) (layer "B.Cu") (net 12))
+  (segment (start 132.92604 89.5) (end 132.325 89.5) (width 0.1) (layer "B.Cu") (net 12))
+  (segment (start 138.7 94.077592) (end 134.632592 94.077592) (width 0.1) (layer "B.Cu") (net 12))
+  (segment (start 134.632592 94.077592) (end 132.96 92.405) (width 0.1) (layer "B.Cu") (net 12))
   (segment (start 144.1196 97.4852) (end 144.1196 97.434245) (width 0.15) (layer "F.Cu") (net 13))
   (segment (start 144.1196 97.434245) (end 142.1 95.414645) (width 0.15) (layer "F.Cu") (net 13))
@@
   (segment (start 146.7 88.718701) (end 146.7 87.107) (width 0.1) (layer "F.Cu") (net 57))
   (zone (net 1) (net_name "GND") (layer "B.Cu") (hatch edge 0.5)
-    (connect_pads (clearance 0.5))
-    (min_thickness 0.25) (filled_areas_thickness no)
-    (fill yes (thermal_gap 0.5) (thermal_bridge_width 0.5) (island_removal_mode 1) (island_area_min 10))
+    (connect_pads (clearance 0.2))
+    (min_thickness 0.2) (filled_areas_thickness no)
+    (fill yes (thermal_gap 0.2) (thermal_bridge_width 0.25) (island_removal_mode 1) (island_area_min 10))
     (polygon
       (pts

Commit message: Add files via upload
Parts:
- added D1: LED, LED_SMD:LED_0603_1608Metric, F.Cu at (147.3, 84.7)
- added G***: LOGO, drawings:cute, B.Cu at (138.8, 98.9)
- added J10: Conn_01x04, Connector_PinHeader_1.00mm:PinHeader_1x04_P1.00mm_Vertical, F.Cu at (150.6, 76.8)
- added R8: 10K, Resistor_SMD:R_0402_1005Metric, F.Cu at (133.6, 88.5)
- added R9: 1K, Resistor_SMD:R_0402_1005Metric, F.Cu at (147.7, 86.8)
- added U1: W25Q128JVS, Package_DFN_QFN:DFN-8-1EP_3x2mm_P0.5mm_EP1.3x1.5mm, F.Cu at (134.2, 82.8)
- J2: value Conn_01x02_Pin -> Conn_01x02
- R6: footprint Resistor_SMD:R_0402_1005Metric -> Resistor_SMD:R_0201_0603Metric
- Y1: footprint Crystal2:Crystal_2.0mm_2.5mm -> Crystal:Crystal_SMD_3225-4Pin_3.2x2.5mm
- moved J9 16.2 mm to (147.9, 95.1), turned to -90 degrees
- moved C7 11.7 mm to (147.3, 93.1), turned to 180 degrees
- moved C1 9.38 mm to (140.1, 84.8), turned to 135 degrees
- moved C2 8.02 mm to (138.1, 76.7), turned to 90 degrees
- moved C12 6.63 mm to (146.6, 98.8)
- moved C11 4.41 mm to (146.6, 99.3), turned to 180 degrees
- moved C14 3.00 mm to (133.1, 77.6)
- moved J8 2.80 mm to (133.2, 96.5)
- moved C16 2.79 mm to (144.8, 99.2), turned to -45 degrees
- moved U5 2.66 mm to (135.5, 76.2), turned to 180 degrees
- moved J7 2.14 mm to (133.2, 98.9)
- moved U2 1.96 mm to (135.3, 83.0)
- moved C9 1.88 mm to (137.5, 89.0), turned to 0 degrees
- moved C8 1.56 mm to (137.5, 93.7), turned to 45 degrees
- moved R6 1.44 mm to (142.5, 96.4), turned to 180 degrees
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Connections:
- net D+ renamed /D+
- net D- renamed /D-
- net Net-(J6-Pin_2) renamed /SWD
- net Net-(J6-Pin_3) renamed /SWCLK
- net Net-(J9-Pin_2) renamed /RST
- net Net-(U3-XIN) renamed /XIN
- net Net-(U3-XOUT) renamed /XOUT
- U3 pad 19: unconnected-(U3-TESTEN-Pad19) -> GND
Routing:
- net +3.3V: track 66.6 -> 80.0 mm, vias 0 -> 2
- net +1V1: track 9.13 -> 22.2 mm, vias 0 -> 2
- net VBUS: track 36.3 -> 48.0 mm
- net /D+: track 4.31 -> 15.7 mm, vias 0 -> 1
- net /RST: track 14.7 -> 3.31 mm, vias 1 -> 0
- net /D-: track 4.18 -> 14.4 mm, vias 0 -> 1
- net /QSPI_SD2: track 6.26 -> 10.8 mm
- net GND: track 42.2 -> 45.9 mm
- net /QSPI_SS: track 9.16 -> 11.8 mm
- net /QSPI_SD1: track 7.13 -> 9.40 mm
- net Net-(D1-K): track 0.00 -> 1.79 mm
- net Net-(C16-Pad1): track 4.67 -> 3.27 mm
- net /QSPI_CLK: track 16.1 -> 17.1 mm
- net /QSPI_SD3: track 17.9 -> 18.6 mm
- net Net-(J4-Pin_3): track 16.8 -> 17.5 mm
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- added copper zone on F.Cu, net +3.3V
Other:
- board size 21.2 x 29.1 mm -> 19.9 x 29 mm
- board text added: "+"
- board text added: "-"
- board text added: "0"
- board text added: "1"
- board text added: "10"
- board text added: "11"
- board text added: "12"
- board text added: "13"
- board text added: "14"
- board text added: "15"
- board text added: "16"
- board text added: "17"
- board text added: "18"
- board text added: "19"
- board text added: "2"
- board text added: "20"
- board text added: "21"
- board text added: "22"
- board text added: "23"
- board text added: "24"
- board text added: "25"
- board text added: "26"
- board text added: "27"
- board text added: "28"
- board text added: "29"
- board text added: "3"
- board text added: "3V3"
- board text added: "4"
- board text added: "5"
- board text added: "5V"
- board text added: "6"
- board text added: "7"
- board text added: "8"
- board text added: "9"
- board text added: "BOOT"
- board text added: "C"
- board text added: "D"
- board text added: "G"
- board text added: "Proto2040 By Treble v1"
- board text added: "RST"
